File: Hardware/antenna_analyzer_rev7.sch (EAGLE design)
At the start: 40 parts, among them J1 DC_JACK, P1 SOLDER_PAD_35_HOLE, P2 SOLDER_PAD_35_HOLE, P3 SOLDER_PAD_35_HOLE, U1 ARDUINO_PRO_MICRO, U2 AD9850_MOD, U3 6002_OP_AMP, U5 SWITCHING_REGULATOR

Commit message: 4X6UB Modifications
Parts:
- removed C5: 10uf, resistor:CPOL-USE1.8-4
- removed CON1: (no value), srs_lib_4:BNC-SMALL
- removed J1: DC_JACK, srs_lib_2:DC_JACK
- removed LCD1: LCD_2_16, srs_lib_4:LCD_2_16
- removed R13: 10, adafruit:R-US_0207/10
- removed R14, R16, R17: 10k, adafruit:R-US_0207/10
- removed R15: 649, adafruit:R-US_0207/10
- removed R18: (no value), Discrete:R-POTENTIOMETER-3362U
- removed S1: RESET, switch-omron:10-XX
- removed S2: MODE, switch-omron:10-XX
- removed S3: BAND, switch-omron:10-XX
- removed U5: SWITCHING_REGULATOR, srs_new:SWITCHING_REGULATOR
- added EXP1, EXP2: (no value), con-lstb:MA05-2
- added JMP1: 0R-JUMPA, jump-0r-smd:0R-JUMPA
- added JP1: (no value), pinhead:PINHD-1X4
- added JP2: (no value), pinhead:PINHD-1X2
- added JP3: (no value), adafruit:PINHD-1X3
- added PAD1: (no value), wirepad:1,6/0,9
- added X1: 1-227161-0, con-coax:1-227161-0
Connections:
- removed net AUX: P2.1, U1.10
- removed net BAND_SEL: R17.1, S3.P, S3.P1, U1.20
- removed net MODE_SEL: R16.1, S2.P, S2.P1, U1.19
- removed net N$12: S1.P, S1.P1, U1.22
- removed net N$37: LCD1.15, R13.1
- removed net N$40: LCD1.3, R14.1, R15.1, R18.3
- removed net TONE: P1.1, U1.9
- new net BEEPER: EXP1.1, JMP1-0R.2
- new net KILL: EXP2.10
- new net N$8: JMP1-0R.3, P2.1, U1.2
- new net POWER_EN: JP1.4, JP3.2
- new net SD_DETECT: EXP2.7
- new net SD_MISO: EXP2.1
- new net SD_MOSI: EXP2.6
- new net SD_SCLK: EXP2.2
- new net SD_SS: EXP2.4
- new net SW_BTN: EXP1.2, U1.20
- new net SW_E1: EXP2.5, U1.11
- new net SW_E2: EXP2.3, U1.12
- new net SW_RST: EXP2.8, U1.9
- net +5V: now also EXP1.10, JP1.2; no longer LCD1.2, R13.2, R14.2, R16.2, R17.2, R18.2, U5.OUT
- net DGND: now also EXP1.9, EXP2.9, JP1.3, JP3.3, PAD1.P, X1.2; no longer C5.-, CON1.G1, CON1.G2, CON1.G3, CON1.G4, J1.1, LCD1.1, LCD1.10, LCD1.16, LCD1.5, LCD1.7, LCD1.8, LCD1.9, R15.2, R18.1, S1.S, S1.S1, S2.S, S2.S1, S3.S, U5.GND
- net LCD_D4: now also EXP1.5; no longer LCD1.11
- net LCD_D5: now also EXP1.6; no longer LCD1.12
- net LCD_D6: now also EXP1.7; no longer LCD1.13
- net LCD_D7: now also EXP1.8; no longer LCD1.14
- net LCD_E: now also EXP1.3, U1.10; no longer LCD1.6, U1.12
- net LCD_RS: now also EXP1.4, U1.19; no longer LCD1.4, U1.11
- net N$1: now also JMP1-0R.1, P1.1, U1.1; no longer C5.+, J1.3, U5.IN
- net N$7: now also X1.1; no longer CON1.CENTER
Other:
- moved on the sheet: P1, P2, U1
